Commit message: update joint limit parameters

File: aliengo_description/xacro/const.xacro (robot description, xacro)
@@ -31,14 +31,14 @@
     <xacro:property name="damping" value="0"/>
     <xacro:property name="friction" value="0"/>
-    <xacro:property name="hip_max" value="70"/>
-    <xacro:property name="hip_min" value="-70"/>
-    <xacro:property name="hip_velocity_max" value="40"/>
-    <xacro:property name="hip_torque_max" value="44.4"/>
-    <xacro:property name="thigh_velocity_max" value="40"/>
-    <xacro:property name="thigh_torque_max" value="44.4"/>
-    <xacro:property name="calf_max" value="-37"/>
-    <xacro:property name="calf_min" value="-159"/>
-    <xacro:property name="calf_velocity_max" value="40"/>
-    <xacro:property name="calf_torque_max" value="44.4"/>
+    <xacro:property name="hip_position_max" value="${70*PI/180.0}"/>
+    <xacro:property name="hip_position_min" value="${-70*PI/180.0}"/>
+    <xacro:property name="hip_velocity_max" value="20"/>
+    <xacro:property name="hip_torque_max" value="44"/>
+    <xacro:property name="thigh_velocity_max" value="20"/>
+    <xacro:property name="thigh_torque_max" value="44"/>
+    <xacro:property name="calf_position_max" value="${-37*PI/180.0}"/>
+    <xacro:property name="calf_position_min" value="${-159*PI/180.0}"/>
+    <xacro:property name="calf_velocity_max" value="16"/>
+    <xacro:property name="calf_torque_max" value="55"/>
     <!-- dynamics inertial value -->
     <!-- trunk -->

File: aliengo_description/xacro/leg.xacro (robot description, xacro)
@@ -10,8 +10,8 @@
             <dynamics damping="${damping}" friction="${friction}"/>
             <xacro:if value="${(mirror_dae == 'true')}">
-                <limit effort="${hip_torque_max}" velocity="${hip_velocity_max}" lower="${hip_min*PI/180.0}" upper="${hip_max*PI/180.0}"/>
+                <limit effort="${hip_torque_max}" velocity="${hip_velocity_max}" lower="${hip_position_min}" upper="${hip_position_max}"/>
             </xacro:if>
             <xacro:if value="${(mirror_dae == 'false')}">
-                <limit effort="${hip_torque_max}" velocity="${hip_velocity_max}" lower="${-hip_max*PI/180.0}" upper="${-hip_min*PI/180.0}"/>
+                <limit effort="${hip_torque_max}" velocity="${hip_velocity_max}" lower="${-hip_position_max}" upper="${-hip_position_min}"/>
             </xacro:if>
         </joint>
@@ -106,5 +106,5 @@
             <axis xyz="0 1 0"/>
             <dynamics damping="${damping}" friction="${friction}"/>
-            <limit effort="${calf_torque_max}" velocity="${calf_velocity_max}" lower="${calf_min*PI/180.0}" upper="${calf_max*PI/180.0}"/>
+            <limit effort="${calf_torque_max}" velocity="${calf_velocity_max}" lower="${calf_position_min}" upper="${calf_position_max}"/>
         </joint>
         <link name="${name}_calf">
