Commit message: fixed the leg bug under Ubuntu18, ROS melodic

File: aliengo_description/xacro/leg.xacro (robot description, xacro)
@@ -9,8 +9,8 @@
             <axis xyz="1 0 0"/>
             <dynamics damping="${damping}" friction="${friction}"/>
-            <xacro:if value="${(mirror_dae == 'true')}">
+            <xacro:if value="${(mirror_dae == True)}">
                 <limit effort="${hip_torque_max}" velocity="${hip_velocity_max}" lower="${hip_position_min}" upper="${hip_position_max}"/>
             </xacro:if>
-            <xacro:if value="${(mirror_dae == 'false')}">
+            <xacro:if value="${(mirror_dae == False)}">
                 <limit effort="${hip_torque_max}" velocity="${hip_velocity_max}" lower="${-hip_position_max}" upper="${-hip_position_min}"/>
             </xacro:if>
@@ -18,14 +18,14 @@
         <link name="${name}_hip">
             <visual>
-                <xacro:if value="${(mirror_dae == 'true') and (front_hind_dae == 'true')}">
+                <xacro:if value="${(mirror_dae == True) and (front_hind_dae == True)}">
                     <origin rpy="0 0 0" xyz="0 0 0"/>
                 </xacro:if>
-                <xacro:if value="${(mirror_dae == 'false') and (front_hind_dae == 'true')}">
+                <xacro:if value="${(mirror_dae == False) and (front_hind_dae == True)}">
                     <origin rpy="${PI} 0 0" xyz="0 0 0"/>
                 </xacro:if>
-                <xacro:if value="${(mirror_dae == 'true') and (front_hind_dae == 'false')}">
+                <xacro:if value="${(mirror_dae == True) and (front_hind_dae == False)}">
                     <origin rpy="0 ${PI} 0" xyz="0 0 0"/>
                 </xacro:if>
-                <xacro:if value="${(mirror_dae == 'false') and (front_hind_dae == 'false')}">
+                <xacro:if value="${(mirror_dae == False) and (front_hind_dae == False)}">
                     <origin rpy="${PI} ${PI} 0" xyz="0 0 0"/>
                 </xacro:if>
@@ -76,8 +76,8 @@
                 <origin rpy="0 0 0" xyz="0 0 0"/>
                 <geometry>
-                    <xacro:if value="${mirror_dae == 'true'}">
+                    <xacro:if value="${mirror_dae == True}">
                         <mesh filename="package://aliengo_description/meshes/thigh.dae" scale="1 1 1"/>
                     </xacro:if>
-                    <xacro:if value="${mirror_dae == 'false'}">
+                    <xacro:if value="${mirror_dae == False}">
                         <mesh filename="package://aliengo_description/meshes/thigh_mirror.dae" scale="1 1 1"/>
                     </xacro:if>

File: aliengo_description/xacro/robot.xacro (robot description, xacro)
@@ -5,7 +5,7 @@
     <xacro:include filename="$(find aliengo_description)/xacro/leg.xacro"/>
     <!-- <xacro:include filename="$(find aliengo_gazebo)/launch/gazebo.xacro"/> -->
-    <!-- Rollover Protection mode will add an additional stick on the top, use "true" or "false" to switch it. -->
-    <xacro:property name="rolloverProtection" value="false"/>
-    <!-- Debug mode will hung up the robot, use "true" or "false" to switch it. -->
+    <!-- Rollover Protection mode will add an additional stick on the top, use "True" or "False" to switch it. -->
+    <xacro:property name="rolloverProtection" value="False"/>
+    <!-- Debug mode will hung up the robot, use "True" or "False" to switch it. -->
     <!-- <xacro:if value="$(arg DEBUG)">
         <link name="world"/>
@@ -58,5 +58,5 @@
         </inertial>
     </link>
-    <xacro:if value="${(rolloverProtection == 'true')}">
+    <xacro:if value="${(rolloverProtection == 'True')}">
         <joint name="stick_joint" type="fixed">
             <parent link="trunk"/>
@@ -112,14 +112,14 @@
         </collision>
     </link>
-    <xacro:leg name="FR" mirror="-1" mirror_dae="false" front_hind="1" front_hind_dae="true">
+    <xacro:leg name="FR" mirror="-1" mirror_dae="False" front_hind="1" front_hind_dae="True">
         <origin rpy="0 0 0" xyz="${leg_offset_x} ${-leg_offset_y} 0"/>
     </xacro:leg>
-    <xacro:leg name="FL" mirror="1" mirror_dae="true" front_hind="1" front_hind_dae="true">
+    <xacro:leg name="FL" mirror="1" mirror_dae="True" front_hind="1" front_hind_dae="True">
         <origin rpy="0 0 0" xyz="${leg_offset_x} ${leg_offset_y} 0"/>
     </xacro:leg>
-    <xacro:leg name="RR" mirror="-1" mirror_dae="false" front_hind="-1" front_hind_dae="false">
+    <xacro:leg name="RR" mirror="-1" mirror_dae="False" front_hind="-1" front_hind_dae="False">
         <origin rpy="0 0 0" xyz="${-leg_offset_x} ${-leg_offset_y} 0"/>
     </xacro:leg>
-    <xacro:leg name="RL" mirror="1" mirror_dae="true" front_hind="-1" front_hind_dae="false">
+    <xacro:leg name="RL" mirror="1" mirror_dae="True" front_hind="-1" front_hind_dae="False">
         <origin rpy="0 0 0" xyz="${-leg_offset_x} ${leg_offset_y} 0"/>
     </xacro:leg>
